File: Eagle/PIC 16F877A Board/PIC 16F877A Board_V4.brd (EAGLE design)
At the start: 127 x 75 mm, 46 parts, among them IC1 7805TV, IC2 LD117AV33, U1 CH340G, Y1 4MHz, Y2 12MHz

Commit message: Modify the footprints of some of the components and modify the drill size of the vias to be more compatable with being made at home
Parts:
- moved R2 1.35 mm to (107.5, 21.9)
- moved RST 1.35 mm to (100.4, 21.9)
Routing:
- net GND: track 173.6 -> 154.7 mm
- net RB7/PGD: track 141.7 -> 144.0 mm
- net RD7/PSP7: track 31.6 -> 29.3 mm
- net RD6/PSP6: track 31.1 -> 29.0 mm
- net RB6/PGC: track 132.2 -> 133.8 mm
- net RD4/PSP4: track 30.3 -> 28.8 mm
- net RD5/PSP5: track 30.5 -> 29.0 mm
- net +V: track 131.3 -> 132.1 mm
