File: Eagle/PIC 16F877A Board/PIC 16F877A Board_V4.brd (EAGLE design)
At the start: 127 x 75 mm, 46 parts, among them IC1 7805TV, IC2 LD117AV33, U1 CH340G, Y1 4MHz, Y2 12MHz

Commit message: Upload modified and old files.
Parts:
- added RXJ, TXJ: (no value), jumper:SJW
- added U$4: (no value), Logos:OMAR_ELSOBKEY_X1_P
- C1, C10, C11: device SparkFun-Capacitors:CAP-PTH-2.54 -> rcl:C025-025X050
- J2: value (none) -> 61729-1011
- ON/OFF: value (none) -> PVA2R
- R1, R2, R3, R4, R5, R6, R7: device SparkFun-Resistors:AXIAL-0.3 -> SparkFun-Resistors:1206
- U$1: value PIC16F877A-I/P -> (none); device PIC - 16F877A:16F877A -> PIC:PDIP-40
- moved U$2 0.62 mm to (75.4, 40.1)
- flipped R1 to the bottom, turned to 0 degrees
- flipped R2 to the bottom
- flipped R3 to the bottom, turned to 180 degrees
- flipped R4 to the bottom, turned to 0 degrees
- flipped R5 to the bottom, turned to 180 degrees
- flipped R6 to the bottom, turned to 180 degrees
- flipped R7 to the bottom, turned to 180 degrees
Connections:
- removed net RC6/TX: PORTC.7, R6.P$2, TX.K, U$1.25
- removed net RC7/RX: PORTC.8, R7.P$2, RX.K, U$1.26
- new net RX0: R7.2, RX.K, RXJ.2
- new net RXC: PORTC.8, RXJ.1, U$1.26
- new net TX0: R6.2, TX.K, TXJ.2
- new net TXC: PORTC.7, TXJ.1, U$1.25
- net +5V: now also R1.2, R2.2, R3.2, R5.2; no longer R1.P$2, R2.P$2, R3.P$2, R5.P$2
- net 3V3: now also R4.2; no longer R4.P$2
- net N$1: now also R4.1; no longer R4.P$1
- net N$2: now also R3.1; no longer R3.P$1
- net N$3: now also R5.1; no longer R5.P$1
- net N$4: now also R1.1; no longer R1.P$1
- net RESET: now also R2.1; no longer R2.P$1
- net RX: now also R6.1; no longer R6.P$1
- net TX: now also R7.1; no longer R7.P$1
Routing:
- net GND: track 154.7 -> 480.6 mm
- net RC7/RX: track 86.3 -> 0.00 mm
- net RC6/TX: track 71.3 -> 0.00 mm
- net TXC: track 0.00 -> 66.6 mm
- net RXC: track 0.00 -> 66.6 mm
- net RX0: track 0.00 -> 20.0 mm, vias 0 -> 2
- net DTR: track 46.7 -> 26.9 mm, vias 0 -> 2
- net TX0: track 0.00 -> 11.8 mm
- net 3V3: track 117.5 -> 127.0 mm, vias 0 -> 2
- net +5V: track 307.4 -> 298.9 mm, vias 10 -> 12
- net TX: track 24.1 -> 26.5 mm
- net RX: track 17.1 -> 18.9 mm
- net RESET: track 117.0 -> 115.8 mm
- net N$4: track 6.03 -> 5.03 mm
- net N$3: track 6.60 -> 5.60 mm
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