File: Eagle/PIC 16F877A Board/PIC 16F877A Board_V4 (SMD).brd (EAGLE design)
At the start: 100 x 60 mm, 48 parts, among them U1 CH340G, U2 AMS1117-5.0, U3 AMS1117-3.3, Y1 4MHz, Y2 12MHz

Commit message: Upload modified and old files.
Parts:
- C1, C10: device SparkFun-Capacitors:CAP-PTH-2.54 -> Capacitor:CAPC2012X110
- C11: value 103 -> 10nF; device SparkFun-Capacitors:CAP-PTH-2.54 -> Capacitor:CAPC2012X110
- C14, C2, C3, C4, C5, C6, C7, C8: device rcl:C025-025X050 -> Capacitor:CAPC2012X110
- R1, R4: value 1k -> (none)
- R2: value 10k -> (none)
- R3, R5, R6, R7: value 1k -> 10k
- U$1: value PIC16F877A-I/P -> (none); device PIC - 16F877A:16F877A -> PIC:PDIP-40
- moved C6 6.26 mm to (44.8, 26.3), turned to 180 degrees
- moved C9 1.88 mm to (62.1, 45.1)
- moved C10 0.85 mm to (22.1, 30.4), turned to 90 degrees
- moved C1 0.83 mm to (17.3, 30.4), turned to 90 degrees
- moved J1 0.73 mm to (10.9, 7.88)
- moved J2 0.18 mm to (10.3, 50.3)
- moved C5 0.12 mm to (62.1, 40.2)
- moved C3 0.12 mm to (76.0, 32.5), turned to 270 degrees
- moved C4 0.12 mm to (71.2, 32.5), turned to 270 degrees
Routing:
- net GND: track 121.4 -> 145.4 mm, vias 7 -> 168
- net RB3/PGM: track 107.0 -> 102.2 mm
- net RESET: track 115.8 -> 111.2 mm
- net XO: track 27.0 -> 23.4 mm
- net D+: track 17.4 -> 14.3 mm
- net D-: track 12.4 -> 9.90 mm
- net DTR: track 8.21 -> 10.4 mm
- net +5V: track 206.6 -> 204.7 mm
- net OSC2: track 12.2 -> 10.9 mm
- net OSC1: track 11.3 -> 9.94 mm
- net RB7/PGD: track 120.7 -> 119.5 mm
- net RB6/PGC: track 107.5 -> 106.5 mm
- net 3V3: track 106.7 -> 107.7 mm
- net RC3/SCK/SCL: track 51.7 -> 50.7 mm
- net RX: track 18.3 -> 17.5 mm
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