File: Eagle/PIC 16F877A Board/PIC 16F877A Board_V4 (SMD).sch (EAGLE design)
At the start: 44 parts, among them J2 61729-1011, U1 CH340G, U2 AMS1117-5.0, U3 AMS1117-3.3, Y1 4MHz, Y2 12MHz

Commit message: Upload modified and old files.
Parts:
- C1, C10: device SparkFun-Capacitors:22PF-PTH-2.54MM-200V-5% -> Capacitor:C_CHIP-0805(2012-METRIC)
- C11: value 103 -> 10nF; device SparkFun-Capacitors:22PF-PTH-2.54MM-200V-5% -> Capacitor:C_CHIP-0805(2012-METRIC)
- C14, C2, C3, C4, C5, C6, C7, C8: device rcl:C-EU025-025X050 -> Capacitor:C_CHIP-0805(2012-METRIC)
- R1, R4: value 1k -> (none)
- R2: value 10k -> (none)
- R3, R5, R6, R7: value 1k -> 10k
- U$1: value PIC16F877A-I/P -> (none); device PIC - 16F877A:PIC16F877A-I/P -> PIC:PIC16F877A-I/P
Other:
- moved on the sheet: C1, C10, C11
