File: Eagle/PIC 16F877A Board/PIC 16F877A Board_V4.sch (EAGLE design)
At the start: 44 parts, among them IC1 7805TV, IC2 LD117AV33, J2 61729-1011, U1 CH340G, Y1 4MHz, Y2 12MHz

Commit message: Upload modified and old files.
Parts:
- added RXJ, TXJ: (no value), jumper:SJW
- C1, C10, C11: device SparkFun-Capacitors:22PF-PTH-2.54MM-200V-5% -> rcl:C-EU025-025X050
- R1, R2, R3, R4, R5, R6, R7: device SparkFun-Resistors:RESISTORAXIAL-0.3 -> SparkFun-Resistors:RESISTOR1206
- U$1: value PIC16F877A-I/P -> (none); device PIC - 16F877A:PIC16F877A-I/P -> PIC:PIC16F877A-I/P
Connections:
- removed net RC6/TX: PORTC.7, R6.2, TX.C, U$1.RC6/TX/CK
- removed net RC7/RX: PORTC.8, R7.2, RX.C, U$1.RC7/RX/DT
- new net RX0: R7.2, RX.C, RXJ.2
- new net RXC: PORTC.8, RXJ.1, U$1.RC7/RX/DT
- new net TX0: R6.2, TX.C, TXJ.2
- new net TXC: PORTC.7, TXJ.1, U$1.RC6/TX/CK
Other:
- moved on the sheet: C1, C10, C11, R3, R6, R7, TX
