File: Eagle/Power Supply/+(3.3, 5, 9, 12)/+(3.3, 5, 9, 12).brd (EAGLE design)
At the start: 150 x 150 mm, 43 parts, among them IC1 7812, IC2 7812, IC3 7812, IC4 7809, IC5 7809, IC6 7809, IC7 7805, IC8 7805, IC9 7805

Commit message: Finish routing.
Parts:
- removed C2: 2200 µF, Wurth_Capacitors_WCAP-ATG8:WCAP-ATG8_16X25(DXL)
- removed S1: ON/OFF, switch-misc:PVA2R
- added 3.3, VCC: (no value), led:LED5MM
- added 3.3V: (no value), pinhead:2X05
- added D19, D20, D21, D22, D23, D24, D25: 1N4004, diode:DO41-10
- added IC10, IC11, IC12: LD117AV33, v-reg:TO220L1
- added J1: (no value), con-jack:SPC4077
- added ON/OFF: (no value), switch-misc:PVA2R
- added R4: 680, SparkFun-Resistors:AXIAL-0.3
- added R5: 100, SparkFun-Resistors:AXIAL-0.3
- added U$1: (no value), Logos:OMAR_ELSOBKEY_X0.5_T
- added U$2, U$3: (no value), Logos:OMAR_ELSOBKEY_X0.5_TN
- 12, 5, 9: device led:LED3MM -> led:LED5MM
- moved 5V 353.1 mm to (97.8, 40.6), turned to 270 degrees
- moved 9V 333.0 mm to (97.8, 25.4), turned to 270 degrees
- moved 12V 313.2 mm to (97.8, 10.2), turned to 270 degrees
- moved 5 309.0 mm to (34.3, 40.6), turned to 270 degrees
- moved D18 307.7 mm to (90.2, 40.6), turned to 90 degrees
- moved D17 299.3 mm to (85.1, 40.6), turned to 90 degrees
- moved R3 294.4 mm to (29.2, 40.6), turned to 90 degrees
- moved 9 290.5 mm to (34.3, 25.4), turned to 270 degrees
- moved D16 287.1 mm to (72.4, 40.6), turned to 90 degrees
- moved D15 278.7 mm to (67.3, 40.6), turned to 90 degrees
- moved R2 276.5 mm to (29.2, 25.4), turned to 90 degrees
- moved 12 272.3 mm to (34.3, 10.2), turned to 270 degrees
- moved D14 266.8 mm to (54.6, 40.6), turned to 90 degrees
- moved D12 260.9 mm to (90.2, 25.4), turned to 90 degrees
- moved R1 258.7 mm to (29.2, 10.2), turned to 90 degrees
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Connections:
- new net +3V3: 3.3V.1, 3.3V.3, 3.3V.5, 3.3V.7, 3.3V.9, D20.C, D22.C, D24.C, R5.P$1
- new net N$27: D22.A, IC11.2
- new net N$28: D23.A, IC11.1
- new net N$29: D24.A, IC12.2
- new net N$3: 3.3.A, R5.P$2
- new net N$30: D25.A, IC12.1
- new net N$31: D20.A, IC10.2
- new net N$4: R4.P$2, VCC.A
- new net N$5: D21.A, IC10.1
- net +5V: now also IC10.3, IC11.3, IC12.3
- net +V: now also ON/OFF.3; no longer S1.3
- net AC: no longer C2.1
- net DC: now also DC.2, J1.3; no longer DC.1
- net GND: now also 3.3.K, 3.3V.10, 3.3V.2, 3.3V.4, 3.3V.6, 3.3V.8, D19.A, D21.C, D23.C, D25.C, DC.1, J1.1, J1.2, ON/OFF.4, ON/OFF.5, VCC.K; no longer C2.2, DC.2, S1.4, S1.5
- net VCC: now also D19.C, ON/OFF.2, R4.P$1; no longer S1.2
Routing:
- net +5V: track 0.00 -> 149.5 mm
- net +12V: track 0.00 -> 145.4 mm, vias 0 -> 2
- net +9V: track 0.00 -> 145.1 mm, vias 0 -> 2
- net VCC: track 0.00 -> 102.3 mm
- net +3V3: track 0.00 -> 89.4 mm
- net GND: track 0.00 -> 81.2 mm, vias 0 -> 12
- net +V: track 0.00 -> 36.8 mm
- net DC: track 0.00 -> 32.8 mm
- net AC: track 0.00 -> 23.2 mm
- net N$1: track 0.00 -> 16.1 mm
- net N$27: track 0.00 -> 12.3 mm
- net N$9: track 0.00 -> 12.3 mm
- net N$15: track 0.00 -> 12.3 mm
- net N$21: track 0.00 -> 12.3 mm
- net N$31: track 0.00 -> 12.3 mm
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Other:
- board size 150 x 150 mm -> 102.9 x 68.2 mm
