File: Eagle/Power Supply/+(3.3, 5, 9, 12)/+(3.3, 5, 9, 12).sch (EAGLE design)
At the start: 43 parts, among them IC1 7812, IC2 7812, IC3 7812, IC4 7809, IC5 7809, IC6 7809, IC7 7805, IC8 7805, IC9 7805

Commit message: Finish routing.
Parts:
- removed C2: 2200 µF, Wurth_Capacitors_WCAP-ATG8:WCAP-ATG8_16X25_860010580021
- removed S1: ON/OFF, switch-misc:PVA2R
- added 3.3, VCC: (no value), led:LED5MM
- added 3.3V: (no value), pinhead:PINHD-2X5
- added D19, D20, D21, D22, D23, D24, D25: 1N4004, diode:1N4004
- added IC10, IC11, IC12: LD117AV33, v-reg:LD117AV33
- added J1: (no value), con-jack:JACK-PLUG0
- added ON/OFF: PVA2R, switch-misc:PVA2R
- added R4: 680, SparkFun-Resistors:RESISTORAXIAL-0.3
- added R5: 100, SparkFun-Resistors:RESISTORAXIAL-0.3
- 12, 5, 9: device led:LED3MM -> led:LED5MM
Connections:
- new net +3V3: 3.3V.1, 3.3V.3, 3.3V.5, 3.3V.7, 3.3V.9, D20.C, D22.C, D24.C, R5.1
- new net N$27: D22.A, IC11.OUT
- new net N$28: D23.A, IC11.ADJ
- new net N$29: D24.A, IC12.OUT
- new net N$3: 3.3.A, R5.2
- new net N$30: D25.A, IC12.ADJ
- new net N$31: D20.A, IC10.OUT
- new net N$4: R4.2, VCC.A
- new net N$5: D21.A, IC10.ADJ
- net +5V: now also IC10.IN, IC11.IN, IC12.IN
- net +V: now also ON/OFF1.P; no longer S11.P
- net AC: no longer C2.+
- net DC: now also DC-2.KL, J1.3; no longer DC-1.KL
- net GND: now also 3.3.C, 3.3V.10, 3.3V.2, 3.3V.4, 3.3V.6, 3.3V.8, D19.A, D21.C, D23.C, D25.C, DC-1.KL, J1.1, J1.2, ON/OFF2.P, ON/OFF2.S, VCC.C; no longer C2.-, DC-2.KL, S12.P, S12.S
- net VCC: now also D19.C, ON/OFF1.S, R4.1; no longer S11.S
Other:
- note added: "AC Input With Rectifying Bridge and Smoothing Capacitros"
- note added: "DC Input"
- note added: "Designed By: Omar Elsobkey @ 13 June 2021"
- note added: "Indicating Leds"
- note added: "Input AC or DC"
- note added: "Output Pins"
- note added: "Regulation"
- note added: "Switch ON/OFF"
- moved on the sheet: 12, 12V, 5, 5V, 9, 9V, AC-1, AC-2, B1, C1, D1, D10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
